Commit message: [Beetle][hand] succeeded to construct urdf/gazebo.xacro files

File: robots/beetle/robots/beetle_hand.gazebo.xacro (robot description, xacro)
@@ -3,5 +3,5 @@
     xmlns:xacro="http://www.ros.org/wiki/xacro" name="beetle" >
   <xacro:arg name="robot_name" default="beetle" />
-  <xacro:include filename="$(find beetle)/urdf/beetle_hand.urdf.xacro" />
+  <xacro:include filename="$(find beetle)/robots/beetle_hand.urdf.xacro" />
   <!-- gazebo plugin for default controller and sensors -->
   <xacro:include filename="$(find aerial_robot_simulation)/xacro/spinal.gazebo.xacro" />

File: robots/beetle/urdf/beetle_hand.urdf.xacro (robot description, xacro)
@@ -200,43 +200,3 @@
     </transmission>
   </xacro:macro>
-  ## beetle hand
-  ## link
-  <link name="handbase">
-    <inertial>
-      <origin xyz="0.0 0.0 0.0" rpy="0 0 0"/>
-      <mass value="0.00001"/>
-      <inertia
-          ixx="0.00001" iyy="0.00001" izz="0.00001"
-          ixy="0.0" ixz="0.0" iyz="0.0"/>
-    </inertial>
-  </link>
-  <link name="hand">
-    <inertial>
-      <origin xyz="0.19178 0.000005 0.025771"/>
-      <mass value="0.3900000"/>
-      <inertia
-  	  ixx="0.000699" ixy="-0.000004" ixz="0.000769"
-  	  iyy="0.005953" iyz="-0.000005"
-  	  izz="0.00541"/>
-    </inertial>
-    <visual>
-      <origin xyz="0 0 0" rpy="0 -1.570796 0"/>
-      <geometry>
-  	<mesh filename="package://beetle/urdf/mesh/beetle_hand_handmech_all.dae"/>
-      </geometry>
-    </visual>
-    <collision>
-      <origin xyz="0.01215 0 0.022" rpy="0 0 0"/>
-      <geometry>
-  	<box size="0.283 0.071 0.118"/>
-      </geometry>
-    </collision>
-  </link>
-  ## beetle hand joint
-  <joint name="handbase_hand_joint" type="fixed">
-    <child link="hand"/>
-    <parent link="handbase"/>
-    <origin xyz="0.031 0 0.107" rpy="0 0 0"/>
-    <axis xyz="1 0 0"/>
-  </joint>
 </robot>
