Commit message: [Beetle_hand] modified urdf for dual hand

File: robots/beetle/robots/beetle_hand.urdf.xacro (robot description, xacro)
@@ -43,5 +43,5 @@
       <origin xyz="0 0 0" rpy="0 0 0"/>
       <geometry>
-        <box size="0.04 0.04 0.04"/>
+        <box size="0.01 0.01 0.01"/>
       </geometry>
     </collision>
@@ -58,5 +58,5 @@
     <inertial>
       <mass value = "0.001" />
-      <origin xyz="0.0 0 0" rpy="0 0 0"/>
+      <origin xyz="0 0 0" rpy="0 0 0"/>
       <inertia
           ixx="0.0001" ixy="0.0000" ixz="0.0000"
@@ -66,5 +66,5 @@
       <origin xyz="0 0 0" rpy="0 0 0"/>
       <geometry>
-        <box size="0.04 0.04 0.04"/>
+        <box size="0.01 0.01 0.01"/>
       </geometry>
     </collision>
@@ -72,5 +72,5 @@
       <origin xyz="0 0 0" rpy="0.0 0 0"/>
       <geometry>
-        <box size="0.04 0.04 0.04"/>
+        <box size="0.01 0.01 0.01"/>
       </geometry>
     </visual>
@@ -154,4 +154,26 @@
     </collision>
   </link>
+  <link name="hand_2">
+    <inertial>
+      <origin xyz="0.19178 0.000005 0.025771"/>
+      <mass value="0.3900000"/>
+      <inertia
+  	  ixx="0.000699" ixy="-0.000004" ixz="0.000769"
+  	  iyy="0.005953" iyz="-0.000005"
+  	  izz="0.00541"/>
+    </inertial>
+    <visual>
+      <origin xyz="0 0 0" rpy="0 0 0"/>
+      <geometry>
+    	<mesh filename="package://beetle/urdf/mesh/beetle_hand_handmech_all.dae"/>
+      </geometry>
+    </visual>
+    <collision>
+      <origin xyz="0.01215 0 0.022" rpy="0 0 0"/>
+      <geometry>
+  	<box size="0.283 0.071 0.118"/>
+      </geometry>
+    </collision>
+  </link>
   ## beetle hand joint
   <joint name="handbase_baselink_joint" type="fixed">
@@ -167,3 +189,9 @@
     <axis xyz="1 0 0"/>
   </joint>
+  <joint name="handbase_hand_joint_2" type="fixed">
+    <child link="hand_2"/>
+    <parent link="handbase"/>
+    <origin xyz="-0.031 0 0.107" rpy="0 0 3.1415"/>
+    <axis xyz="1 0 0"/>
+  </joint>
 </robot>

Commit message: [Beetle_hand] modified urdf for dual hand

File: robots/beetle/robots/beetle_hand.urdf.xacro (robot description, xacro)
@@ -192,5 +192,5 @@
     <child link="hand_2"/>
     <parent link="handbase"/>
-    <origin xyz="-0.031 0 0.107" rpy="0 0 3.1415"/>
+    <origin xyz="-0.031 0 0.107" rpy="0 0 3.141"/>
     <axis xyz="1 0 0"/>
   </joint>

Commit message: [Beetle_hand] modified urdf for dual hand

File: robots/beetle/robots/beetle_hand.urdf.xacro (robot description, xacro)
@@ -192,5 +192,5 @@
     <child link="hand_2"/>
     <parent link="handbase"/>
-    <origin xyz="-0.031 0 0.107" rpy="0 0 3.141"/>
+    <origin xyz="-0.031 0 0.107" rpy="0 0 3.1415"/>
     <axis xyz="1 0 0"/>
   </joint>
