Commit message: [Gryllo] Successed for 1 revolute joint, but not for more than 2

File: robots/gryllo/urdf/gryllo/gryllo_detailed.urdf.xacro (robot description, xacro)
@@ -33,7 +33,7 @@
       </visual>
       <collision>
-	<origin xyz="0 0 0" rpy="0 0 0"/>
-	<geometry>
-	  <box size="0.25 0.25 0.10"/>
+	<origin xyz="-0.05 0 0" rpy="0 0 0"/>
+	<geometry>
+	  <box size="0.25 0.25 0.20"/>
 	</geometry>
       </collision>
@@ -54,7 +54,7 @@
       </visual>
       <collision>
-	<origin xyz="0 0 0" rpy="0 0 0"/>
-	<geometry>
-	  <box size="0.25 0.25 0.10"/>
+	<origin xyz="-0.050 0 0" rpy="0 0 0"/>
+	<geometry>
+	  <box size="0.25 0.25 0.20"/>
 	</geometry>
       </collision>
@@ -64,7 +64,7 @@
     <link name="act_unit">
       <inertial>
-        <origin xyz="0.0099 -0.0655 0.0012" rpy="0 0 0"/>
+        <origin xyz="0.1251 0.0001 -0.0184" rpy="0 0 0"/>
         <mass value="0.30623"/>
-        <inertia ixx="0.00169" iyy="0.00221" izz="0.00065" ixy="0.00000" ixz="-0.00008" iyz="0.00000"/>
+        <inertia ixx="0.00048" iyy="0.00576" izz="0.00542" ixy="0.00001" ixz="-0.00078" iyz="0.00000"/>
       </inertial>
       <visual>
@@ -101,5 +101,5 @@
       <parent link="act_unit"/>
       <child link="fc"/>
-      <origin xyz="0 0 0" rpy="0 0 0"/>
+      <origin xyz="0.11520 0.00001 0.04759" rpy="0 0 0"/>
     </joint>
     #### spine links 1-5 ####
@@ -176,13 +176,66 @@
     ## joints ##
     #### spine joints ####
-    <joint name="spine_joint_1" type="revolute">
+    <!-- <joint name="spine_joint_1" type="revolute"> -->
+    <!--   <parent link="act_unit"/> -->
+    <!--   <child link="spine_1"/> -->
+    <!--   <origin xyz="0.19432 0.0 0.01373" rpy="0 0 0"/> -->
+    <!--   <axis xyz="0 0 1"/> -->
+    <!--   <limit lower="-0.52" upper="0.52" effort="5.0" velocity="2.0"/> -->
+    <!--   <dynamics damping="10.0" friction="0.0"/> -->
+    <!-- </joint> -->
+    <!-- <joint name="spine_joint_2" type="revolute"> -->
+    <!--   <parent link="spine_1"/> -->
+    <!--   <child link="spine_2"/> -->
+    <!--   <origin xyz="${pitch} 0 0" rpy="0 0 0"/> -->
+    <!--   <axis xyz="0 0 1"/> -->
+    <!--   <limit lower="-0.52" upper="0.52" effort="5.0" velocity="2.0"/> -->
+    <!--   <dynamics damping="10.0" friction="0.0"/> -->
+    <!--   <mimic joint="spine_joint_1" multiplier="1.0" offset="0.0"/> -->
+    <!-- </joint> -->
+    <joint name="spine_joint_3" type="revolute">
+      <parent link="spine_2"/>
+      <child link="spine_3"/>
+      <origin xyz="${pitch} 0 0" rpy="0 0 0"/>
+      <axis xyz="0 0 1"/>
+      <limit lower="-0.52" upper="0.52" effort="5.0" velocity="2.0"/>
+      <dynamics damping="20.0" friction="2.0"/>
+      <mimic joint="spine_joint_1" multiplier="1.0" offset="0.0"/>
+    </joint>
+    <!-- <joint name="spine_joint_4" type="revolute"> -->
+    <!--   <parent link="spine_3"/> -->
+    <!--   <child link="spine_4"/> -->
+    <!--   <origin xyz="${pitch} 0 0" rpy="0 0 0"/> -->
+    <!--   <axis xyz="0 0 1"/> -->
+    <!--   <limit lower="-0.52" upper="0.52" effort="5.0" velocity="2.0"/> -->
+    <!--   <dynamics damping="10.0" friction="0.0"/> -->
+    <!--   <mimic joint="spine_joint_1" multiplier="1.0" offset="0.0"/> -->
+    <!-- </joint> -->
+    <joint name="spine_joint_5" type="revolute">
+      <parent link="spine_4"/>
+      <child link="spine_5"/>
+      <origin xyz="${pitch} 0 0" rpy="0 0 0"/>
+      <axis xyz="0 0 1"/>
+      <limit lower="-0.52" upper="0.52" effort="5.0" velocity="2.0"/>
+      <dynamics damping="10.0" friction="0.0"/>
+      <mimic joint="spine_joint_1" multiplier="1.0" offset="0.0"/>
+    </joint>
+    <!-- <joint name="spine_joint_6" type="revolute"> -->
+    <!--   <parent link="spine_5"/> -->
+    <!--   <child link="act_unit_2"/> -->
+    <!--   <origin xyz="${pitch} 0 0" rpy="0 0 0"/> -->
+    <!--   <axis xyz="0 0 1"/> -->
+    <!--   <limit lower="-0.52" upper="0.52" effort="5.0" velocity="2.0"/> -->
+    <!--   <dynamics damping="10.0" friction="0.0"/> -->
+    <!--   <mimic joint="spine_joint_1" multiplier="1.0" offset="0.0"/> -->
+    <!-- </joint> -->
+    <joint name="spine_joint_1" type="fixed">
       <parent link="act_unit"/>
       <child link="spine_1"/>
-      <origin xyz="0.079 0.001 -0.033" rpy="0 0 0"/>
+      <origin xyz="0.19432 0.0 0.01373" rpy="0 0 0"/>
       <axis xyz="0 0 1"/>
       <limit lower="-0.52" upper="0.52" effort="5.0" velocity="2.0"/>
       <dynamics damping="1.0" friction="0.0"/>
     </joint>
-    <joint name="spine_joint_2" type="revolute">
+    <joint name="spine_joint_2" type="fixed">
       <parent link="spine_1"/>
       <child link="spine_2"/>
@@ -192,44 +245,4 @@
       <dynamics damping="1.0" friction="0.0"/>
     </joint>
-    <joint name="spine_joint_3" type="revolute">
-      <parent link="spine_2"/>
-      <child link="spine_3"/>
-      <origin xyz="${pitch} 0 0" rpy="0 0 0"/>
-      <axis xyz="0 0 1"/>
-      <limit lower="-0.52" upper="0.52" effort="5.0" velocity="2.0"/>
-      <dynamics damping="1.0" friction="0.0"/>
-    </joint>
-    <joint name="spine_joint_4" type="revolute">
-      <parent link="spine_3"/>
-      <child link="spine_4"/>
-      <origin xyz="${pitch} 0 0" rpy="0 0 0"/>
-      <axis xyz="0 0 1"/>
-      <limit lower="-0.52" upper="0.52" effort="5.0" velocity="2.0"/>
-      <dynamics damping="1.0" friction="0.0"/>
-    </joint>
-    <joint name="spine_joint_5" type="revolute">
-      <parent link="spine_4"/>
-      <child link="spine_5"/>
-      <origin xyz="${pitch} 0 0" rpy="0 0 0"/>
-      <axis xyz="0 0 1"/>
-      <limit lower="-0.52" upper="0.52" effort="5.0" velocity="2.0"/>
-      <dynamics damping="1.0" friction="0.0"/>
-    </joint>
-    <!-- <joint name="spine_joint_1" type="fixed"> -->
-    <!--   <parent link="act_unit"/> -->
-    <!--   <child link="spine_1"/> -->
-    <!--   <origin xyz="0.079 0.001 -0.033" rpy="0 0 0"/> -->
-    <!--   <axis xyz="0 0 1"/> -->
-    <!--   <limit lower="-0.52" upper="0.52" effort="5.0" velocity="2.0"/> -->
-    <!--   <dynamics damping="1.0" friction="0.0"/> -->
-    <!-- </joint> -->
-    <!-- <joint name="spine_joint_2" type="fixed"> -->
-    <!--   <parent link="spine_1"/> -->
-    <!--   <child link="spine_2"/> -->
-    <!--   <origin xyz="${pitch} 0 0" rpy="0 0 0"/> -->
-    <!--   <axis xyz="0 0 1"/> -->
-    <!--   <limit lower="-0.52" upper="0.52" effort="5.0" velocity="2.0"/> -->
-    <!--   <dynamics damping="1.0" friction="0.0"/> -->
-    <!-- </joint> -->
     <!-- <joint name="spine_joint_3" type="fixed"> -->
     <!--   <parent link="spine_2"/> -->
@@ -240,12 +253,12 @@
     <!--   <dynamics damping="1.0" friction="0.0"/> -->
     <!-- </joint> -->
-    <!-- <joint name="spine_joint_4" type="fixed"> -->
-    <!--   <parent link="spine_3"/> -->
-    <!--   <child link="spine_4"/> -->
-    <!--   <origin xyz="${pitch} 0 0" rpy="0 0 0"/> -->
-    <!--   <axis xyz="0 0 1"/> -->
-    <!--   <limit lower="-0.52" upper="0.52" effort="5.0" velocity="2.0"/> -->
-    <!--   <dynamics damping="1.0" friction="0.0"/> -->
-    <!-- </joint> -->
+    <joint name="spine_joint_4" type="fixed">
+      <parent link="spine_3"/>
+      <child link="spine_4"/>
+      <origin xyz="${pitch} 0 0" rpy="0 0 0"/>
+      <axis xyz="0 0 1"/>
+      <limit lower="-0.52" upper="0.52" effort="5.0" velocity="2.0"/>
+      <dynamics damping="1.0" friction="0.0"/>
+    </joint>
     <!-- <joint name="spine_joint_5" type="fixed"> -->
     <!--   <parent link="spine_4"/> -->
@@ -264,4 +277,65 @@
       <dynamics damping="1.0" friction="0.0"/>
     </joint>
+    #### transmissions ####
+    <!-- <transmission name="spine_tran_1"> -->
+    <!--   <type>transmission_interface/SimpleTransmission</type> -->
+    <!--   <joint name="spine_joint_1"> -->
+    <!-- 	<hardwareInterface>hardware_interface/EffortJointInterface</hardwareInterface> -->
+    <!--   </joint> -->
+    <!--   <actuator name="spine_servo_1"> -->
+    <!-- 	<hardwareInterface>hardware_interface/EffortJointInterface</hardwareInterface> -->
+    <!-- 	<mechanicalReduction>1</mechanicalReduction> -->
+    <!--   </actuator> -->
+    <!-- </transmission> -->
+    <!-- <transmission name="spine_tran_2"> -->
+    <!--   <type>transmission_interface/SimpleTransmission</type> -->
+    <!--   <joint name="spine_joint_2"> -->
+    <!-- 	<hardwareInterface>hardware_interface/EffortJointInterface</hardwareInterface> -->
+    <!--   </joint> -->
+    <!--   <actuator name="spine_servo_2"> -->
+    <!-- 	<hardwareInterface>hardware_interface/EffortJointInterface</hardwareInterface> -->
+    <!-- 	<mechanicalReduction>1</mechanicalReduction> -->
+    <!--   </actuator> -->
+    <!-- </transmission> -->
+    <transmission name="spine_tran_3">
+      <type>transmission_interface/SimpleTransmission</type>
+      <joint name="spine_joint_3">
+	<hardwareInterface>hardware_interface/EffortJointInterface</hardwareInterface>
+      </joint>
+      <actuator name="spine_servo_3">
+	<hardwareInterface>hardware_interface/EffortJointInterface</hardwareInterface>
+	<mechanicalReduction>1</mechanicalReduction>
+      </actuator>
+    </transmission>
+    <!-- <transmission name="spine_tran_4"> -->
+    <!--   <type>transmission_interface/SimpleTransmission</type> -->
+    <!--   <joint name="spine_joint_4"> -->
+    <!-- 	<hardwareInterface>hardware_interface/EffortJointInterface</hardwareInterface> -->
+    <!--   </joint> -->
+    <!--   <actuator name="spine_servo_4"> -->
+    <!-- 	<hardwareInterface>hardware_interface/EffortJointInterface</hardwareInterface> -->
+    <!-- 	<mechanicalReduction>1</mechanicalReduction> -->
+    <!--   </actuator> -->
+    <!-- </transmission> -->
+    <transmission name="spine_tran_5">
+      <type>transmission_interface/SimpleTransmission</type>
+      <joint name="spine_joint_5">
+	<hardwareInterface>hardware_interface/EffortJointInterface</hardwareInterface>
+      </joint>
+      <actuator name="spine_servo_5">
+	<hardwareInterface>hardware_interface/EffortJointInterface</hardwareInterface>
+	<mechanicalReduction>1</mechanicalReduction>
+      </actuator>
+    </transmission>
+    <!-- <transmission name="spine_tran_6"> -->
+    <!--   <type>transmission_interface/SimpleTransmission</type> -->
+    <!--   <joint name="spine_joint_6"> -->
+    <!-- 	<hardwareInterface>hardware_interface/EffortJointInterface</hardwareInterface> -->
+    <!--   </joint> -->
+    <!--   <actuator name="spine_servo_6"> -->
+    <!-- 	<hardwareInterface>hardware_interface/EffortJointInterface</hardwareInterface> -->
+    <!-- 	<mechanicalReduction>1</mechanicalReduction> -->
+    <!--   </actuator> -->
+    <!-- </transmission> -->
     #### rotor arms ####
     <link name="rotor_arm${child1}">
@@ -320,5 +394,5 @@
       <parent link="base_link"/>
       <child link="act_unit"/>
-      <origin rpy="0 0 0" xyz="0.115 0.001 0.047"/>
+      <origin rpy="0 0 0" xyz="0.0 0.0 0.0"/>
       <axis xyz="1 0 0"/>
       <dynamics damping="0.8" friction="0.0"/>
@@ -338,5 +412,5 @@
       <parent link="act_unit_2"/>
       <child link="base_link_2"/>
-      <origin rpy="0 0 0" xyz="0.194 0.0 -0.014"/>
+      <origin rpy="0 0 0" xyz="0.195 0.0 -0.014"/>
       <axis xyz="1 0 0"/>
       <dynamics damping="0.8" friction="0.0"/>

Commit message: [Gryllo] last commit was a little broken

File: robots/gryllo/urdf/gryllo/gryllo_detailed.urdf.xacro (robot description, xacro)
@@ -211,13 +211,13 @@
     <!--   <mimic joint="spine_joint_1" multiplier="1.0" offset="0.0"/> -->
     <!-- </joint> -->
-    <joint name="spine_joint_5" type="revolute">
-      <parent link="spine_4"/>
-      <child link="spine_5"/>
-      <origin xyz="${pitch} 0 0" rpy="0 0 0"/>
-      <axis xyz="0 0 1"/>
-      <limit lower="-0.52" upper="0.52" effort="5.0" velocity="2.0"/>
-      <dynamics damping="10.0" friction="0.0"/>
-      <mimic joint="spine_joint_1" multiplier="1.0" offset="0.0"/>
-    </joint>
+    <!-- <joint name="spine_joint_5" type="revolute"> -->
+    <!--   <parent link="spine_4"/> -->
+    <!--   <child link="spine_5"/> -->
+    <!--   <origin xyz="${pitch} 0 0" rpy="0 0 0"/> -->
+    <!--   <axis xyz="0 0 1"/> -->
+    <!--   <limit lower="-0.52" upper="0.52" effort="5.0" velocity="2.0"/> -->
+    <!--   <dynamics damping="10.0" friction="0.0"/> -->
+    <!--   <mimic joint="spine_joint_1" multiplier="1.0" offset="0.0"/> -->
+    <!-- </joint> -->
     <!-- <joint name="spine_joint_6" type="revolute"> -->
     <!--   <parent link="spine_5"/> -->
@@ -261,12 +261,12 @@
       <dynamics damping="1.0" friction="0.0"/>
     </joint>
-    <!-- <joint name="spine_joint_5" type="fixed"> -->
-    <!--   <parent link="spine_4"/> -->
-    <!--   <child link="spine_5"/> -->
-    <!--   <origin xyz="${pitch} 0 0" rpy="0 0 0"/> -->
-    <!--   <axis xyz="0 0 1"/> -->
-    <!--   <limit lower="-0.52" upper="0.52" effort="5.0" velocity="2.0"/> -->
-    <!--   <dynamics damping="1.0" friction="0.0"/> -->
-    <!-- </joint> -->
+    <joint name="spine_joint_5" type="fixed">
+      <parent link="spine_4"/>
+      <child link="spine_5"/>
+      <origin xyz="${pitch} 0 0" rpy="0 0 0"/>
+      <axis xyz="0 0 1"/>
+      <limit lower="-0.52" upper="0.52" effort="5.0" velocity="2.0"/>
+      <dynamics damping="1.0" friction="0.0"/>
+    </joint>
     <joint name="spine_joint_6" type="fixed">
       <parent link="spine_5"/>
@@ -318,14 +318,14 @@
     <!--   </actuator> -->
     <!-- </transmission> -->
-    <transmission name="spine_tran_5">
-      <type>transmission_interface/SimpleTransmission</type>
-      <joint name="spine_joint_5">
-	<hardwareInterface>hardware_interface/EffortJointInterface</hardwareInterface>
-      </joint>
-      <actuator name="spine_servo_5">
-	<hardwareInterface>hardware_interface/EffortJointInterface</hardwareInterface>
-	<mechanicalReduction>1</mechanicalReduction>
-      </actuator>
-    </transmission>
+    <!-- <transmission name="spine_tran_5"> -->
+    <!--   <type>transmission_interface/SimpleTransmission</type> -->
+    <!--   <joint name="spine_joint_5"> -->
+    <!-- 	<hardwareInterface>hardware_interface/EffortJointInterface</hardwareInterface> -->
+    <!--   </joint> -->
+    <!--   <actuator name="spine_servo_5"> -->
+    <!-- 	<hardwareInterface>hardware_interface/EffortJointInterface</hardwareInterface> -->
+    <!-- 	<mechanicalReduction>1</mechanicalReduction> -->
+    <!--   </actuator> -->
+    <!-- </transmission> -->
     <!-- <transmission name="spine_tran_6"> -->
     <!--   <type>transmission_interface/SimpleTransmission</type> -->
