Commit message: [Gryllo] all spine joints can get initial pose, no gazebo tragedy

File: robots/gryllo/urdf/gryllo/gryllo_detailed.urdf.xacro (robot description, xacro)
@@ -176,21 +176,21 @@
     ## joints ##
     #### spine joints ####
-    <!-- <joint name="spine_joint_1" type="revolute"> -->
-    <!--   <parent link="act_unit"/> -->
-    <!--   <child link="spine_1"/> -->
-    <!--   <origin xyz="0.19432 0.0 0.01373" rpy="0 0 0"/> -->
-    <!--   <axis xyz="0 0 1"/> -->
-    <!--   <limit lower="-0.52" upper="0.52" effort="5.0" velocity="2.0"/> -->
-    <!--   <dynamics damping="10.0" friction="0.0"/> -->
-    <!-- </joint> -->
-    <!-- <joint name="spine_joint_2" type="revolute"> -->
-    <!--   <parent link="spine_1"/> -->
-    <!--   <child link="spine_2"/> -->
-    <!--   <origin xyz="${pitch} 0 0" rpy="0 0 0"/> -->
-    <!--   <axis xyz="0 0 1"/> -->
-    <!--   <limit lower="-0.52" upper="0.52" effort="5.0" velocity="2.0"/> -->
-    <!--   <dynamics damping="10.0" friction="0.0"/> -->
-    <!--   <mimic joint="spine_joint_1" multiplier="1.0" offset="0.0"/> -->
-    <!-- </joint> -->
+    <joint name="spine_joint_1" type="revolute">
+      <parent link="act_unit"/>
+      <child link="spine_1"/>
+      <origin xyz="0.19432 0.0 0.01373" rpy="0 0 0"/>
+      <axis xyz="0 0 1"/>
+      <limit lower="-0.52" upper="0.52" effort="5.0" velocity="2.0"/>
+      <dynamics damping="10.0" friction="0.0"/>
+    </joint>
+    <joint name="spine_joint_2" type="revolute">
+      <parent link="spine_1"/>
+      <child link="spine_2"/>
+      <origin xyz="${pitch} 0 0" rpy="0 0 0"/>
+      <axis xyz="0 0 1"/>
+      <limit lower="-0.52" upper="0.52" effort="5.0" velocity="2.0"/>
+      <dynamics damping="10.0" friction="0.0"/>
+      <mimic joint="spine_joint_1" multiplier="1.0" offset="0.0"/>
+    </joint>
     <joint name="spine_joint_3" type="revolute">
       <parent link="spine_2"/>
@@ -202,56 +202,5 @@
       <mimic joint="spine_joint_1" multiplier="1.0" offset="0.0"/>
     </joint>
-    <!-- <joint name="spine_joint_4" type="revolute"> -->
-    <!--   <parent link="spine_3"/> -->
-    <!--   <child link="spine_4"/> -->
-    <!--   <origin xyz="${pitch} 0 0" rpy="0 0 0"/> -->
-    <!--   <axis xyz="0 0 1"/> -->
-    <!--   <limit lower="-0.52" upper="0.52" effort="5.0" velocity="2.0"/> -->
-    <!--   <dynamics damping="10.0" friction="0.0"/> -->
-    <!--   <mimic joint="spine_joint_1" multiplier="1.0" offset="0.0"/> -->
-    <!-- </joint> -->
-    <!-- <joint name="spine_joint_5" type="revolute"> -->
-    <!--   <parent link="spine_4"/> -->
-    <!--   <child link="spine_5"/> -->
-    <!--   <origin xyz="${pitch} 0 0" rpy="0 0 0"/> -->
-    <!--   <axis xyz="0 0 1"/> -->
-    <!--   <limit lower="-0.52" upper="0.52" effort="5.0" velocity="2.0"/> -->
-    <!--   <dynamics damping="10.0" friction="0.0"/> -->
-    <!--   <mimic joint="spine_joint_1" multiplier="1.0" offset="0.0"/> -->
-    <!-- </joint> -->
-    <!-- <joint name="spine_joint_6" type="revolute"> -->
-    <!--   <parent link="spine_5"/> -->
-    <!--   <child link="act_unit_2"/> -->
-    <!--   <origin xyz="${pitch} 0 0" rpy="0 0 0"/> -->
-    <!--   <axis xyz="0 0 1"/> -->
-    <!--   <limit lower="-0.52" upper="0.52" effort="5.0" velocity="2.0"/> -->
-    <!--   <dynamics damping="10.0" friction="0.0"/> -->
-    <!--   <mimic joint="spine_joint_1" multiplier="1.0" offset="0.0"/> -->
-    <!-- </joint> -->
-    <joint name="spine_joint_1" type="fixed">
-      <parent link="act_unit"/>
-      <child link="spine_1"/>
-      <origin xyz="0.19432 0.0 0.01373" rpy="0 0 0"/>
-      <axis xyz="0 0 1"/>
-      <limit lower="-0.52" upper="0.52" effort="5.0" velocity="2.0"/>
-      <dynamics damping="1.0" friction="0.0"/>
-    </joint>
-    <joint name="spine_joint_2" type="fixed">
-      <parent link="spine_1"/>
-      <child link="spine_2"/>
-      <origin xyz="${pitch} 0 0" rpy="0 0 0"/>
-      <axis xyz="0 0 1"/>
-      <limit lower="-0.52" upper="0.52" effort="5.0" velocity="2.0"/>
-      <dynamics damping="1.0" friction="0.0"/>
-    </joint>
-    <!-- <joint name="spine_joint_3" type="fixed"> -->
-    <!--   <parent link="spine_2"/> -->
-    <!--   <child link="spine_3"/> -->
-    <!--   <origin xyz="${pitch} 0 0" rpy="0 0 0"/> -->
-    <!--   <axis xyz="0 0 1"/> -->
-    <!--   <limit lower="-0.52" upper="0.52" effort="5.0" velocity="2.0"/> -->
-    <!--   <dynamics damping="1.0" friction="0.0"/> -->
-    <!-- </joint> -->
-    <joint name="spine_joint_4" type="fixed">
+    <joint name="spine_joint_4" type="revolute">
       <parent link="spine_3"/>
       <child link="spine_4"/>
@@ -259,7 +208,8 @@
       <axis xyz="0 0 1"/>
       <limit lower="-0.52" upper="0.52" effort="5.0" velocity="2.0"/>
-      <dynamics damping="1.0" friction="0.0"/>
-    </joint>
-    <joint name="spine_joint_5" type="fixed">
+      <dynamics damping="10.0" friction="0.0"/>
+      <mimic joint="spine_joint_1" multiplier="1.0" offset="0.0"/>
+    </joint>
+    <joint name="spine_joint_5" type="revolute">
       <parent link="spine_4"/>
       <child link="spine_5"/>
@@ -267,7 +217,8 @@
       <axis xyz="0 0 1"/>
       <limit lower="-0.52" upper="0.52" effort="5.0" velocity="2.0"/>
-      <dynamics damping="1.0" friction="0.0"/>
-    </joint>
-    <joint name="spine_joint_6" type="fixed">
+      <dynamics damping="10.0" friction="0.0"/>
+      <mimic joint="spine_joint_1" multiplier="1.0" offset="0.0"/>
+    </joint>
+    <joint name="spine_joint_6" type="revolute">
       <parent link="spine_5"/>
       <child link="act_unit_2"/>
@@ -275,27 +226,38 @@
       <axis xyz="0 0 1"/>
       <limit lower="-0.52" upper="0.52" effort="5.0" velocity="2.0"/>
-      <dynamics damping="1.0" friction="0.0"/>
+      <dynamics damping="10.0" friction="0.0"/>
+      <mimic joint="spine_joint_1" multiplier="1.0" offset="0.0"/>
     </joint>
     #### transmissions ####
-    <!-- <transmission name="spine_tran_1"> -->
-    <!--   <type>transmission_interface/SimpleTransmission</type> -->
-    <!--   <joint name="spine_joint_1"> -->
-    <!-- 	<hardwareInterface>hardware_interface/EffortJointInterface</hardwareInterface> -->
-    <!--   </joint> -->
-    <!--   <actuator name="spine_servo_1"> -->
-    <!-- 	<hardwareInterface>hardware_interface/EffortJointInterface</hardwareInterface> -->
-    <!-- 	<mechanicalReduction>1</mechanicalReduction> -->
-    <!--   </actuator> -->
-    <!-- </transmission> -->
-    <!-- <transmission name="spine_tran_2"> -->
-    <!--   <type>transmission_interface/SimpleTransmission</type> -->
-    <!--   <joint name="spine_joint_2"> -->
-    <!-- 	<hardwareInterface>hardware_interface/EffortJointInterface</hardwareInterface> -->
-    <!--   </joint> -->
-    <!--   <actuator name="spine_servo_2"> -->
-    <!-- 	<hardwareInterface>hardware_interface/EffortJointInterface</hardwareInterface> -->
-    <!-- 	<mechanicalReduction>1</mechanicalReduction> -->
-    <!--   </actuator> -->
-    <!-- </transmission> -->
+    <transmission name="spine_tran_1">
+      <type>transmission_interface/SimpleTransmission</type>
+      <joint name="spine_joint_1">
+	<hardwareInterface>hardware_interface/EffortJointInterface</hardwareInterface>
+      </joint>
+      <actuator name="spine_servo_1">
+	<hardwareInterface>hardware_interface/EffortJointInterface</hardwareInterface>
+	<mechanicalReduction>1</mechanicalReduction>
+      </actuator>
+    </transmission>
+    <gazebo reference="spine_joint_1">
+      <implicitSpringDamper>true</implicitSpringDamper>
+      <springStiffness>1.0</springStiffness>
+      <springReference>0.0</springReference>
+    </gazebo>
+    <transmission name="spine_tran_2">
+      <type>transmission_interface/SimpleTransmission</type>
+      <joint name="spine_joint_2">
+	<hardwareInterface>hardware_interface/EffortJointInterface</hardwareInterface>
+      </joint>
+      <actuator name="spine_servo_2">
+	<hardwareInterface>hardware_interface/EffortJointInterface</hardwareInterface>
+	<mechanicalReduction>1</mechanicalReduction>
+      </actuator>
+    </transmission>
+    <gazebo reference="spine_joint_2">
+      <implicitSpringDamper>true</implicitSpringDamper>
+      <springStiffness>1.0</springStiffness>
+      <springReference>0.0</springReference>
+    </gazebo>
     <transmission name="spine_tran_3">
       <type>transmission_interface/SimpleTransmission</type>
@@ -308,34 +270,54 @@
       </actuator>
     </transmission>
-    <!-- <transmission name="spine_tran_4"> -->
-    <!--   <type>transmission_interface/SimpleTransmission</type> -->
-    <!--   <joint name="spine_joint_4"> -->
-    <!-- 	<hardwareInterface>hardware_interface/EffortJointInterface</hardwareInterface> -->
-    <!--   </joint> -->
-    <!--   <actuator name="spine_servo_4"> -->
-    <!-- 	<hardwareInterface>hardware_interface/EffortJointInterface</hardwareInterface> -->
-    <!-- 	<mechanicalReduction>1</mechanicalReduction> -->
-    <!--   </actuator> -->
-    <!-- </transmission> -->
-    <!-- <transmission name="spine_tran_5"> -->
-    <!--   <type>transmission_interface/SimpleTransmission</type> -->
-    <!--   <joint name="spine_joint_5"> -->
-    <!-- 	<hardwareInterface>hardware_interface/EffortJointInterface</hardwareInterface> -->
-    <!--   </joint> -->
-    <!--   <actuator name="spine_servo_5"> -->
-    <!-- 	<hardwareInterface>hardware_interface/EffortJointInterface</hardwareInterface> -->
-    <!-- 	<mechanicalReduction>1</mechanicalReduction> -->
-    <!--   </actuator> -->
-    <!-- </transmission> -->
-    <!-- <transmission name="spine_tran_6"> -->
-    <!--   <type>transmission_interface/SimpleTransmission</type> -->
-    <!--   <joint name="spine_joint_6"> -->
-    <!-- 	<hardwareInterface>hardware_interface/EffortJointInterface</hardwareInterface> -->
-    <!--   </joint> -->
-    <!--   <actuator name="spine_servo_6"> -->
-    <!-- 	<hardwareInterface>hardware_interface/EffortJointInterface</hardwareInterface> -->
-    <!-- 	<mechanicalReduction>1</mechanicalReduction> -->
-    <!--   </actuator> -->
-    <!-- </transmission> -->
+    <gazebo reference="spine_joint_3">
+      <implicitSpringDamper>true</implicitSpringDamper>
+      <springStiffness>1.0</springStiffness>
+      <springReference>0.0</springReference>
+    </gazebo>
+    <transmission name="spine_tran_4">
+      <type>transmission_interface/SimpleTransmission</type>
+      <joint name="spine_joint_4">
+	<hardwareInterface>hardware_interface/EffortJointInterface</hardwareInterface>
+      </joint>
+      <actuator name="spine_servo_4">
+	<hardwareInterface>hardware_interface/EffortJointInterface</hardwareInterface>
+	<mechanicalReduction>1</mechanicalReduction>
+      </actuator>
+    </transmission>
+    <gazebo reference="spine_joint_4">
+      <implicitSpringDamper>true</implicitSpringDamper>
+      <springStiffness>1.0</springStiffness>
+      <springReference>0.0</springReference>
+    </gazebo>
+    <transmission name="spine_tran_5">
+      <type>transmission_interface/SimpleTransmission</type>
+      <joint name="spine_joint_5">
+	<hardwareInterface>hardware_interface/EffortJointInterface</hardwareInterface>
+      </joint>
+      <actuator name="spine_servo_5">
+	<hardwareInterface>hardware_interface/EffortJointInterface</hardwareInterface>
+	<mechanicalReduction>1</mechanicalReduction>
+      </actuator>
+    </transmission>
+    <gazebo reference="spine_joint_5">
+      <implicitSpringDamper>true</implicitSpringDamper>
+      <springStiffness>1.0</springStiffness>
+      <springReference>0.0</springReference>
+    </gazebo>
+    <transmission name="spine_tran_6">
+      <type>transmission_interface/SimpleTransmission</type>
+      <joint name="spine_joint_6">
+	<hardwareInterface>hardware_interface/EffortJointInterface</hardwareInterface>
+      </joint>
+      <actuator name="spine_servo_6">
+	<hardwareInterface>hardware_interface/EffortJointInterface</hardwareInterface>
+	<mechanicalReduction>1</mechanicalReduction>
+      </actuator>
+    </transmission>
+    <gazebo reference="spine_joint_6">
+      <implicitSpringDamper>true</implicitSpringDamper>
+      <springStiffness>1.0</springStiffness>
+      <springReference>0.0</springReference>
+    </gazebo>
     #### rotor arms ####
     <link name="rotor_arm${child1}">
