Commit message: [gryllo] Modified fc link, rviz_config

File: robots/gryllo/robots/gryllo/gryllo.urdf.xacro (robot description, xacro)
@@ -1,11 +1,11 @@
 <?xml version="1.0"?>
 <robot
-    xmlns:xacro="http://www.ros.org/wiki/xacro" name="gimbalrotor" >
-  <xacro:include filename="$(find gryllo)/urdf/gryllo/gimbalrotor.urdf.xacro" />
+    xmlns:xacro="http://www.ros.org/wiki/xacro" name="gryllo" >
+  <xacro:include filename="$(find gryllo)/urdf/gryllo/gryllo.urdf.xacro" />
   <xacro:include filename="$(find gryllo)/urdf/gryllo/common.xacro" />
-  <xacro:gimbalrotor_center_link child1="1" child2="2" child3="3" child4="4"/>
-  <xacro:gimbalrotor_thrust_link self="1" rotor_direction="1"/>
-  <xacro:gimbalrotor_thrust_link self="2" rotor_direction="-1"/>
-  <xacro:gimbalrotor_thrust_link self="3" rotor_direction="1"/>
-  <xacro:gimbalrotor_thrust_link self="4" rotor_direction="-1"/>
+  <xacro:gryllo_center_link child1="1" child2="2" child3="3" child4="4"/>
+  <xacro:gryllo_thrust_link self="1" rotor_direction="1"/>
+  <xacro:gryllo_thrust_link self="2" rotor_direction="-1"/>
+  <xacro:gryllo_thrust_link self="3" rotor_direction="1"/>
+  <xacro:gryllo_thrust_link self="4" rotor_direction="-1"/>
 </robot>

File: robots/gryllo/urdf/gryllo/gryllo.urdf.xacro (robot description, xacro)
@@ -1,6 +1,6 @@
 <?xml version="1.0"?>
 <robot
-    xmlns:xacro="http://www.ros.org/wiki/xacro" name="gimbalrotor_link" >
-  <xacro:macro name="gimbalrotor_center_link" params="child1 child2 child3 child4">
+    xmlns:xacro="http://www.ros.org/wiki/xacro" name="gryllo_link" >
+  <xacro:macro name="gryllo_center_link" params="child1 child2 child3 child4">
     ## dummy
     <link name="root">
@@ -25,8 +25,8 @@
         <origin xyz="0.1981 0.0000 0.1105
 " rpy="0 0 0"/>
-        <mass value="1.99364"/>
+        <mass value="2.0000"/>
         <inertia
             ixx="0.03038" iyy="0.25319" izz="0.24155"
-            ixy="0.00001" ixz="0.03528" iyz="0.00001"/>
+            ixy="0.00001" ixz="0.00031" iyz="0.00000"/>
       </inertial>
       <visual>
@@ -37,7 +37,7 @@
       </visual>
       <collision>
-        <origin xyz="0 0 0.09" rpy="0 0 0"/>
-        <geometry>
-          <box size="0.996 0.350 0.180"/>
+        <origin xyz="0.225 0.0 0.1" rpy="0 0 0"/>
+        <geometry>
+          <box size="1.25 0.625 0.183"/>
         </geometry>
       </collision>
@@ -46,5 +46,5 @@
     <link name="fc">
       <inertial>
-        <origin xyz="-0.017 -0.001 0.148" rpy="0 0 0"/>
+        <origin xyz="0.0 0.0 0.0" rpy="0 0 0"/>
         <mass value="0.00001"/>
         <inertia
@@ -57,5 +57,5 @@
       <child link="fc"/>
       <parent link="base_link"/>
-      <origin rpy="0 0 0" xyz="0 0 0"/>
+      <origin xyz="-0.0173 0.0000 0.1476" rpy="0 0 0"/>
       <axis xyz="0 0 1"/>
     </joint>
@@ -70,16 +70,4 @@
             izz="0.0001"/>
       </inertial>
-      <!-- <visual> -->
-      <!--   <origin xyz="0 0 0" rpy="0 0 0"/> -->
-      <!--   <geometry> -->
-      <!--     <mesh filename="package://gimbalrotor/urdf/quad/mesh/rotor_arm.STL"/> -->
-      <!--   </geometry> -->
-      <!-- </visual> -->
-      <!-- <collision> -->
-      <!--   <origin xyz="0 0 0" rpy="0 0 0"/> -->
-      <!--   <geometry> -->
-      <!--     <box size="0.131 0.0325 0.065"/> -->
-      <!--   </geometry> -->
-      <!-- </collision> -->
     </link>
     <joint name="base_arm_joint${child1}" type="fixed">
@@ -98,16 +86,4 @@
             izz="0.0001"/>
       </inertial>
-      <!-- <visual> -->
-      <!--   <origin xyz="0 0 0" rpy="0 0 0"/> -->
-      <!--   <geometry> -->
-      <!--     <mesh filename="package://gimbalrotor/urdf/quad/mesh/rotor_arm.STL"/> -->
-      <!--   </geometry> -->
-      <!-- </visual> -->
-      <!-- <collision> -->
-      <!--   <origin xyz="0 0 0" rpy="0 0 0"/> -->
-      <!--   <geometry> -->
-      <!--     <box size="0.131 0.0325 0.065"/> -->
-      <!--   </geometry>p -->
-      <!-- </collision> -->
     </link>
     <joint name="base_arm_joint${child2}" type="fixed">
@@ -126,16 +102,4 @@
             izz="0.0001"/>
       </inertial>
-      <!-- <visual> -->
-      <!--   <origin xyz="0 0 0" rpy="0 0 0"/> -->
-      <!--   <geometry> -->
-      <!--     <mesh filename="package://gimbalrotor/urdf/quad/mesh/rotor_arm.STL"/> -->
-      <!--   </geometry> -->
-      <!-- </visual> -->
-      <!-- <collision> -->
-      <!--   <origin xyz="0 0 0" rpy="0 0 0"/> -->
-      <!--   <geometry> -->
-      <!--     <box size="0.131 0.0325 0.065"/> -->
-      <!--   </geometry> -->
-      <!-- </collision> -->
     </link>
     <joint name="base_arm_joint${child3}" type="fixed">
@@ -154,16 +118,4 @@
             izz="0.0001"/>
       </inertial>
-      <!-- <visual> -->
-      <!--   <origin xyz="0 0 0" rpy="0 0 0"/> -->
-      <!--   <geometry> -->
-      <!--     <mesh filename="package://gimbalrotor/urdf/quad/mesh/rotor_arm.STL"/> -->
-      <!--   </geometry> -->
-      <!-- </visual> -->
-      <!-- <collision> -->
-      <!--   <origin xyz="0 0 0" rpy="0 0 0"/> -->
-      <!--   <geometry> -->
-      <!--     <box size="0.131 0.0325 0.065"/> -->
-      <!--   </geometry> -->
-      <!-- </collision> -->
     </link>
     <joint name="base_arm_joint${child4}" type="fixed">
@@ -175,5 +127,5 @@
     <xacro:friction self="base_link"/>
   </xacro:macro>
-  <xacro:macro name="gimbalrotor_thrust_link" params="self rotor_direction">
+  <xacro:macro name="gryllo_thrust_link" params="self rotor_direction">
     ## link
     #### rotor parent link (virtual) ####
