Commit message: [gryllo] modified urdf, set correct urdf to the launch.

File: robots/gryllo/robots/gryllo/gryllo.gazebo.xacro (robot description, xacro)
@@ -2,6 +2,6 @@
 <robot
     xmlns:xacro="http://www.ros.org/wiki/xacro" name="gimbalrotor" >
-  <xacro:arg name="robot_name" default="gimbalrotor" />
-  <xacro:include filename="$(find gimbalrotor)/robots/gryllo/gimbalrotor.urdf.xacro" />
+  <xacro:arg name="robot_name" default="gryllo" />
+  <xacro:include filename="$(find gryllo)/robots/gryllo/gryllo.urdf.xacro" />
   <!-- gazebo plugin for default controller and sensors -->
   <xacro:include filename="$(find aerial_robot_simulation)/xacro/spinal.gazebo.xacro" />

File: robots/gryllo/robots/gryllo/gryllo.urdf.xacro (robot description, xacro)
@@ -2,6 +2,6 @@
 <robot
     xmlns:xacro="http://www.ros.org/wiki/xacro" name="gimbalrotor" >
-  <xacro:include filename="$(find gimbalrotor)/urdf/gryllo/gimbalrotor.urdf.xacro" />
-  <xacro:include filename="$(find gimbalrotor)/urdf/gryllo/common.xacro" />
+  <xacro:include filename="$(find gryllo)/urdf/gryllo/gimbalrotor.urdf.xacro" />
+  <xacro:include filename="$(find gryllo)/urdf/gryllo/common.xacro" />
   <xacro:gimbalrotor_center_link child1="1" child2="2" child3="3" child4="4"/>
   <xacro:gimbalrotor_thrust_link self="1" rotor_direction="1"/>

File: robots/gryllo/urdf/gryllo/gimbalrotor.urdf.xacro (robot description, xacro)
@@ -25,5 +25,5 @@
         <origin xyz="0.0267 0.0111 0.0000
 " rpy="0 0 0"/>
-        <mass value="0.1598"/>
+        <mass value="2.0000"/>
         <inertia
             ixx="0.03038" iyy="0.25319" izz="0.24155"

Commit message: [Gryllo] Created rough 'detailed-urdf.'

File: robots/gryllo/robots/gryllo/gryllo.gazebo.xacro (robot description, xacro)
@@ -3,5 +3,6 @@
     xmlns:xacro="http://www.ros.org/wiki/xacro" name="gryllo" >
   <xacro:arg name="robot_name" default="gryllo" />
-  <xacro:include filename="$(find gryllo)/robots/gryllo/gryllo.urdf.xacro" />
+  <!-- <xacro:include filename="$(find gryllo)/robots/gryllo/gryllo.urdf.xacro" /> -->
+  <xacro:include filename="$(find gryllo)/robots/gryllo/gryllo_detailed.urdf.xacro" />
   <!-- gazebo plugin for default controller and sensors -->
   <xacro:include filename="$(find aerial_robot_simulation)/xacro/spinal.gazebo.xacro" />

File: robots/gryllo/robots/gryllo/gryllo.urdf.xacro (robot description, xacro)
@@ -4,4 +4,5 @@
   <xacro:include filename="$(find gryllo)/urdf/gryllo/gryllo.urdf.xacro" />
   <xacro:include filename="$(find gryllo)/urdf/gryllo/common.xacro" />
+  <!-- rotor macro -->
   <xacro:gryllo_center_link child1="1" child2="2" child3="3" child4="4"/>
   <xacro:gryllo_thrust_link self="1" rotor_direction="-1"/>
@@ -9,3 +10,6 @@
   <xacro:gryllo_thrust_link self="3" rotor_direction="-1"/>
   <xacro:gryllo_thrust_link self="4" rotor_direction="1"/>
+  <!-- gryllo spine macro -->
+  <xacro:property name="N" value="5"/>
+  <xacro:property name="pitch" value="0.0605"/>
 </robot>

File: robots/gryllo/urdf/gryllo/gryllo.urdf.xacro (robot description, xacro)
@@ -32,5 +32,5 @@
         <origin xyz="0 0 0" rpy="0 0 0"/>
         <geometry>
-          <mesh filename="package://gryllo/urdf/gryllo/mesh/bodylink_45d.STL"/>
+          <mesh filename="package://gryllo/urdf/gryllo/mesh/simple/bodylink_45d.STL"/>
         </geometry>
       </visual>
@@ -146,5 +146,5 @@
         <origin xyz="0 0 0" rpy="0 0 0"/>
         <geometry>
-          <mesh filename="package://gryllo/urdf/gryllo/mesh/rotor_unit_leftside.STL"/>
+          <mesh filename="package://gryllo/urdf/gryllo/mesh/simple/rotor_unit_leftside.STL"/>
         </geometry>
       </visual>
